Commit message: draft

File: resource/Panda/panda.urdf (robot description, URDF)
Before this commit: robot panda, 12 links, 11 joints
Links:
- added link panda_rightfinger_tip
Joints:
- added joint panda_finger_joint3: type fixed, parent panda_rightfinger, child panda_rightfinger_tip, origin xyz=0 0 0 rpy=0 0 0

Commit message: exercise 1

File: resource/Panda/panda.urdf (robot description, URDF)
Before this commit: robot panda, 13 links, 12 joints
Links:
- added link world
Joints:
- added joint worldTolink1: type fixed, parent world, child panda_link0, origin xyz=0 0 0
- joint panda_finger_joint3: origin xyz=0 0 0 rpy=0 0 0 -> xyz=0 0 0.05 rpy=0 0 0
